File: ZumoRobot.kicad_sch (KiCad schematic)
At the start: 33 parts, among them CN1 B2B-XH-A, CN2 B2B-XH-A, SW1 TS-1088-AR02016, SW2 TS-1088-AR02016, U1 ESP32-S3-WROOM-1

Commit message: change motor driver
Parts:
- removed LED2: XL-1608SURC-06, EasyEDA:LED0603-RD_RED, symbol EasyEDA:XL-1608SURC-06
- removed R8: 10K, PCM_Resistor_SMD_AKL:R_0603_1608Metric, symbol PCM_Resistor_US_AKL:R_0603
- added CN3, CN4: B2B-XH-A, EasyEDA:CONN-TH_B2B-XH-A-LF-SN, symbol EasyEDA:B2B-XH-A
- added J1, J2: Conn_01x04_Socket, EasyEDA:CONN-TH_B4B-PH-K-S, symbol Connector:Conn_01x04_Socket
Connections:
- net +3V3: now also J1.1 (Pin_1), J1.2 (Pin_2), J1.3 (Pin_3), J1.4 (Pin_4)
- net GND: now also J2.1 (Pin_1), J2.2 (Pin_2), J2.3 (Pin_3), J2.4 (Pin_4)
- net PWMA1: now reaches U1.15 (GPIO3/TOUCH3/ADC1_CH2)
- net PWMA2: now reaches U1.16 (GPIO46)
- net PWMB2: now reaches U1.17 (GPIO9/TOUCH9/ADC1_CH8/FSPIHD/SUBSPIHD)
- net PWMB1: now reaches U1.18 (GPIO10/TOUCH10/ADC1_CH9/FSPICS0/FSPIIO4/SUBSPICS0)
- net IN-ToF1: now reaches U1.19 (GPIO11/TOUCH11/ADC2_CH0/FSPID/FSPIIO5/SUBSPID)
- net IN-ToF2: now reaches U1.20 (GPIO12/TOUCH12/ADC2_CH1/FSPICLK/FSPIIO6/SUBSPICLK)
- net IN-ToF3: now reaches U1.21 (GPIO13/TOUCH13/ADC2_CH2/FSPIQ/FSPIIO7/SUBSPIQ)
- net IN-ToF4: now reaches U1.22 (GPIO14/TOUCH14/ADC2_CH3/FSPIWP/FSPIDQS/SUBSPIWP)
- net Motor_Fault: now reaches U1.6 (GPIO6/TOUCH6/ADC1_CH5)
- net +5V renamed VCC
- net SERVO_PWM: no longer names the net of U1.38 (GPIO2/TOUCH2/ADC1_CH1)
- new net DRV8411APWR/M1A: CN3.1
- new net DRV8411APWR/M1B: CN3.2
- new net DRV8411APWR/M2A: CN4.1
- new net DRV8411APWR/M2B: CN4.2
Other:
- removed sheet PH3A_Driver
- removed sheet PH3A_Driver1
- added sheet DRV8411APWR (DRV8411APWR.kicad_sch)
- note removed: "Fuente 5V"
- note removed: "Solo Salida"

Commit message: avances
Parts:
- removed J1, J2: Conn_01x04_Socket, EasyEDA:CONN-TH_B4B-PH-K-S, symbol Connector:Conn_01x04_Socket
- added U4, U5: DB125-3.5-4P-GN, EasyEDA:CONN-TH_DB125-3.5-4P-GN, symbol EasyEDA:DB125-3.5-4P-GN
Connections:
- net +3V3: now also U4.1, U4.2, U4.3, U4.4
- net GND: now also U5.1, U5.2, U5.3, U5.4
