File: ZumoRobot.kicad_sch (KiCad schematic)
At the start: 35 parts, among them CN1 B2B-XH-A, CN2 B2B-XH-A, CN3 B2B-XH-A, CN4 B2B-XH-A, SW1 TS-1088-AR02016, SW2 TS-1088-AR02016, U1 ESP32-S3-WROOM-1, U4 DB125-3.5-4P-GN, U5 DB125-3.5-4P-GN

Commit message: terminada
Parts:
- added IR-1, IR-2, IR-3, IR-4, SCL1, SDA1, X-SHUT1, X-SHUT2, X-SHUT3: TestPoint, PCM_SparkFun-Connector:TestPoint-1.25mm, symbol PCM_4ms_Connector:TestPoint
- added R10, R11: 2.2K, PCM_Resistor_SMD_AKL:R_0603_1608Metric, symbol PCM_Resistor_US_AKL:R_0603
- renumbered R9 to R8, R10 to R9, U4 to U2, U5 to U3
Connections:
- net +3V3: now also R10.2, R11.2
- net X-SHUT 3: now reaches U1.10 (GPIO17/U1TXD/ADC2_CH6)
- net X-SHUT 3: now also X-SHUT2.1
- net IR-1: now reaches U1.11 (GPIO18/U1RXD/ADC2_CH7/CLK_OUT3)
- net IR-1: now also IR-1.1
- net IR-2: now reaches U1.23 (GPIO21)
- net IR-2: now also IR-2.1
- net X-SHUT 4: now reaches U1.24 (GPIO47/SPICLK_P/SUBSPICLK_P_DIFF)
- net IR-4: now reaches U1.26 (GPIO45)
- net IR-4: now also IR-4.1
- net IR-3: now reaches U1.31 (GPIO38/FSPIWP/SUBSPIWP)
- net IR-3: now also IR-3.1
- net IN-ToF1 renamed SDA TOF
- net SDA TOF: now also R10.1, SDA1.1
- net IN-ToF2 renamed SCL TOF
- net SCL TOF: now also R11.1, SCL1.1
- net IN-ToF3 renamed X-SHUT 1 
- net X-SHUT 1 : now also X-SHUT1.1
- net IN-ToF4 renamed X-SHUT 2
- net X-SHUT 2: now also X-SHUT3.1

Commit message: commit final
Parts:
- IR-1, IR-2, IR-3, IR-4, SCL1, SDA1, X-SHUT1, X-SHUT2, X-SHUT3: now left out of the parts list
- U1: LCSC Part (none) -> C2913202
Changed lines of the file:
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@@
 	(text "switch ON/OFF\n"
 		(exclude_from_sim no)
-		(at 25.146 55.372 0)
+		(at 27.432 56.896 0)
 		(effects
 			(font
@@
 	(wire
 		(pts
-			(xy 40.64 44.45) (xy 40.64 46.99)
+			(xy 39.37 48.26) (xy 39.37 46.99)
 		)
 		(stroke
@@
 	(wire
 		(pts
-			(xy 40.64 46.99) (xy 33.02 46.99)
+			(xy 39.37 46.99) (xy 33.02 46.99)
 		)
 		(stroke
@@
 	(symbol
 		(lib_id "power:+7.5V")
-		(at 40.64 44.45 0)
-		(mirror y)
+		(at 39.37 48.26 270)
+		(mirror x)
 		(unit 1)
 		(body_style 1)
@@
 		(fields_autoplaced yes)
 		(property "Reference" "#PWR06"
-			(at 40.64 48.26 0)
+			(at 35.56 48.26 0)
 			(hide yes)
 			(show_name no)
@@
 		)
 		(property "Value" "+7.5V"
-			(at 40.64 39.37 0)
+			(at 43.18 48.26 90)
 			(show_name no)
 			(do_not_autoplace no)
@@
 					(size 1.12 1.12)
 				)
+				(justify left)
 			)
 		)
 		(property "Footprint" ""
-			(at 40.64 44.45 0)
+			(at 39.37 48.26 0)
 			(hide yes)
 			(show_name no)
@@
 		)
 		(property "Datasheet" ""
-			(at 40.64 44.45 0)
+			(at 39.37 48.26 0)
 			(hide yes)
 			(show_name no)
@@
 		)
 		(property "Description" "Power symbol creates a global label with name \"+7.5V\""
-			(at 40.64 44.45 0)
+			(at 39.37 48.26 0)
 			(hide yes)
 			(show_name no)
@@
 		(body_style 1)
 		(exclude_from_sim no)
-		(in_bom yes)
+		(in_bom no)
 		(on_board yes)
 		(in_pos_files yes)
@@
 		(body_style 1)
 		(exclude_from_sim no)
-		(in_bom yes)
+		(in_bom no)
 		(on_board yes)
 		(in_pos_files yes)
@@
 		(body_style 1)
 		(exclude_from_sim no)
-		(in_bom yes)
+		(in_bom no)
 		(on_board yes)
 		(in_pos_files yes)
@@
 		(body_style 1)
 		(exclude_from_sim no)
-		(in_bom yes)
+		(in_bom no)
 		(on_board yes)
 		(in_pos_files yes)
@@
 			)
 		)
+		(property "LCSC Part" "C2913202"
+			(at 222.25 168.91 0)
+			(hide yes)
+			(show_name no)
+			(do_not_autoplace no)
+			(effects
+				(font
+					(size 1.27 1.27)
+				)
+			)
+		)
 		(pin "22"
 		)
@@
 		(body_style 1)
 		(exclude_from_sim no)
-		(in_bom yes)
+		(in_bom no)
 		(on_board yes)
 		(in_pos_files yes)
@@
 		(body_style 1)
 		(exclude_from_sim no)
-		(in_bom yes)
+		(in_bom no)
 		(on_board yes)
 		(in_pos_files yes)
@@
 		(body_style 1)
 		(exclude_from_sim no)
-		(in_bom yes)
+		(in_bom no)
 		(on_board yes)
 		(in_pos_files yes)
@@
 		(body_style 1)
 		(exclude_from_sim no)
-		(in_bom yes)
+		(in_bom no)
 		(on_board yes)
 		(in_pos_files yes)
@@
 		(body_style 1)
 		(exclude_from_sim no)
-		(in_bom yes)
+		(in_bom no)
 		(on_board yes)
 		(in_pos_files yes)
