File: _autosave-ZumoRobot.kicad_sch (KiCad schematic)
At the start: 35 parts, among them CN1 B2B-XH-A, CN2 B2B-XH-A, CN3 B2B-XH-A, CN4 B2B-XH-A, SW1 TS-1088-AR02016, SW2 TS-1088-AR02016, U1 ESP32-S3-WROOM-1, U4 DB125-3.5-4P-GN, U5 DB125-3.5-4P-GN

Commit message: avanzes
Parts:
- added R10, R11: 2.2K, PCM_Resistor_SMD_AKL:R_0603_1608Metric, symbol PCM_Resistor_US_AKL:R_0603
- added SCL1, SDA1, X-SHUT1, X-SHUT2, X-SHUT3, X-SHUT4, X-SHUT5, X-SHUT6: TestPoint, PCM_SparkFun-Connector:TestPoint-1.25mm, symbol PCM_4ms_Connector:TestPoint
- renumbered R9 to R8, R10 to R9, U4 to U2, U5 to U3
Connections:
- net +3V3: now also R10.2, R11.2
- net X-SHUT 3: now reaches U1.10 (GPIO17/U1TXD/ADC2_CH6)
- net X-SHUT 3: now also X-SHUT2.1
- net IR-1: now reaches U1.11 (GPIO18/U1RXD/ADC2_CH7/CLK_OUT3)
- net IR-2: now reaches U1.23 (GPIO21)
- net X-SHUT 4: now reaches U1.24 (GPIO47/SPICLK_P/SUBSPICLK_P_DIFF)
- net X-SHUT 4: now also X-SHUT4.1
- net IR-4: now reaches U1.26 (GPIO45)
- net IR-3: now reaches U1.31 (GPIO38/FSPIWP/SUBSPIWP)
- net IN-ToF1 renamed SDA TOF
- net SDA TOF: now also R10.1, SDA1.1
- net IN-ToF2 renamed SCL TOF
- net SCL TOF: now also R11.1, SCL1.1
- net IN-ToF3 renamed X-SHUT 1 
- net X-SHUT 1 : now also X-SHUT1.1
- net IN-ToF4 renamed X-SHUT 2
- net X-SHUT 2: now also X-SHUT3.1
