File: BuckConverter.kicad_sch (KiCad schematic)
At the start: 7 parts, among them U2 TPS62172DSG

Commit message: change motor driver
Parts:
- renumbered C8 to C7, C11 to C8, R12 to R11
Changed lines of the file:
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@@
 		(dnp no)
 		(fields_autoplaced yes)
-		(property "Reference" "#PWR053"
+		(property "Reference" "#PWR025"
 			(at 203.2 101.6 0)
 			(hide yes)
@@
 			(project "ZumoRobot"
 				(path "/b3437995-bb94-4c2f-9ed8-b1af477fe956/bbae36a6-1608-41fb-8b94-fa07ee9e7141"
-					(reference "#PWR053")
+					(reference "#PWR025")
 					(unit 1)
 				)
@@
 		(in_pos_files yes)
 		(dnp no)
-		(property "Reference" "R12"
+		(property "Reference" "R11"
 			(at 278.13 99.06 90)
 			(show_name no)
@@
 			(project "ZumoRobot"
 				(path "/b3437995-bb94-4c2f-9ed8-b1af477fe956/bbae36a6-1608-41fb-8b94-fa07ee9e7141"
-					(reference "R12")
+					(reference "R11")
 					(unit 1)
 				)
@@
 		(dnp no)
 		(fields_autoplaced yes)
-		(property "Reference" "C11"
+		(property "Reference" "C8"
 			(at 290.83 107.9499 0)
 			(show_name no)
@@
 			(project "ZumoRobot"
 				(path "/b3437995-bb94-4c2f-9ed8-b1af477fe956/bbae36a6-1608-41fb-8b94-fa07ee9e7141"
-					(reference "C11")
+					(reference "C8")
 					(unit 1)
 				)
@@
 		(dnp no)
 		(fields_autoplaced yes)
-		(property "Reference" "#PWR028"
+		(property "Reference" "#PWR026"
 			(at 203.2 139.7 0)
 			(hide yes)
@@
 			(project "ZumoRobot"
 				(path "/b3437995-bb94-4c2f-9ed8-b1af477fe956/bbae36a6-1608-41fb-8b94-fa07ee9e7141"
-					(reference "#PWR028")
+					(reference "#PWR026")
 					(unit 1)
 				)
@@
 		(dnp no)
 		(fields_autoplaced yes)
-		(property "Reference" "#PWR036"
+		(property "Reference" "#PWR029"
 			(at 287.02 123.19 0)
 			(hide yes)
@@
 			(project "ZumoRobot"
 				(path "/b3437995-bb94-4c2f-9ed8-b1af477fe956/bbae36a6-1608-41fb-8b94-fa07ee9e7141"
-					(reference "#PWR036")
+					(reference "#PWR029")
 					(unit 1)
 				)
@@
 		(dnp no)
 		(fields_autoplaced yes)
-		(property "Reference" "#PWR030"
+		(property "Reference" "#PWR027"
 			(at 227.33 129.54 0)
 			(hide yes)
@@
 			(project "ZumoRobot"
 				(path "/b3437995-bb94-4c2f-9ed8-b1af477fe956/bbae36a6-1608-41fb-8b94-fa07ee9e7141"
-					(reference "#PWR030")
+					(reference "#PWR027")
 					(unit 1)
 				)
@@
 		(dnp no)
 		(fields_autoplaced yes)
-		(property "Reference" "#PWR035"
+		(property "Reference" "#PWR028"
 			(at 287.02 82.55 0)
 			(hide yes)
@@
 			(project "ZumoRobot"
 				(path "/b3437995-bb94-4c2f-9ed8-b1af477fe956/bbae36a6-1608-41fb-8b94-fa07ee9e7141"
-					(reference "#PWR035")
+					(reference "#PWR028")
 					(unit 1)
 				)
@@
 		(in_pos_files yes)
 		(dnp no)
-		(property "Reference" "C8"
+		(property "Reference" "C7"
 			(at 199.39 110.4899 0)
 			(show_name no)
@@
 			(project "ZumoRobot"
 				(path "/b3437995-bb94-4c2f-9ed8-b1af477fe956/bbae36a6-1608-41fb-8b94-fa07ee9e7141"
-					(reference "C8")
-					(unit 1)
-				)
+					(reference "C7")
+					(unit 1)
+				)

Commit message: avances
Parts:
- removed L1: MDMK2020T2R2MM, Snapeda:IND_MDMK2020T1R0MM_TAY, symbol Snapeda:MDMK2020T2R2MM
- added L2: LQM2HPN2R2MJ0L, EasyEDA:L1008, symbol EasyEDA:LQM2HPN2R2MJ0L
Connections:
- net L1_3V3: now also L2.1
- net Reg3v3_out: now also L2.2
Changed lines of the file:
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@@
 	(wire
 		(pts
-			(xy 240.03 100.33) (xy 251.46 100.33)
+			(xy 240.03 100.33) (xy 254 100.33)
 		)
 		(stroke
@@
 	(wire
 		(pts
+			(xy 264.16 100.33) (xy 283.21 100.33)
+		)
+		(stroke
+			(width 0.508)
+			(type default)
+		)
+	)
+	(wire
+		(pts
 			(xy 287.02 95.25) (xy 287.02 100.33)
 		)
@@
 		(pts
 			(xy 214.63 100.33) (xy 219.71 100.33)
-		)
-		(stroke
-			(width 0.508)
-			(type default)
-		)
-	)
-	(wire
-		(pts
-			(xy 266.7 100.33) (xy 283.21 100.33)
 		)
 		(stroke
@@
 	)
 	(symbol
+		(lib_id "EasyEDA:LQM2HPN2R2MJ0L")
+		(at 259.08 100.33 0)
+		(unit 1)
+		(body_style 1)
+		(exclude_from_sim no)
+		(in_bom yes)
+		(on_board yes)
+		(in_pos_files yes)
+		(dnp no)
+		(fields_autoplaced yes)
+		(property "Reference" "L2"
+			(at 259.05 93.98 0)
+			(show_name no)
+			(do_not_autoplace no)
+			(effects
+				(font
+					(size 1.27 1.27)
+				)
+			)
+		)
+		(property "Value" "LQM2HPN2R2MJ0L"
+			(at 259.05 96.52 0)
+			(show_name no)
+			(do_not_autoplace no)
+			(effects
+				(font
+					(size 1.27 1.27)
+				)
+			)
+		)
+		(property "Footprint" "EasyEDA:L1008"
+			(at 259.08 107.95 0)
+			(hide yes)
+			(show_name no)
+			(do_not_autoplace no)
+			(effects
+				(font
+					(size 1.27 1.27)
+				)
+			)
+		)
+		(property "Datasheet" "https://lcsc.com/product-detail/Inductors-SMD_muRata_LQM2HPN2R2MJ0L_2-2uH-20-1A_C113101.html"
+			(at 259.08 110.49 0)
+			(hide yes)
+			(show_name no)
+			(do_not_autoplace no)
+			(effects
+				(font
+					(size 1.27 1.27)
+				)
+			)
+		)
+		(property "Description" ""
+			(at 259.08 100.33 0)
+			(hide yes)
+			(show_name no)
+			(do_not_autoplace no)
+			(effects
+				(font
+					(size 1.27 1.27)
+				)
+			)
+		)
+		(property "Manufacturer" "muRata(村田)"
+			(at 259.08 113.03 0)
+			(hide yes)
+			(show_name no)
+			(do_not_autoplace no)
+			(effects
+				(font
+					(size 1.27 1.27)
+				)
+			)
+		)
+		(property "MPN" "LQM2HPN2R2MJ0L"
+			(at 259.08 115.57 0)
+			(hide yes)
+			(show_name no)
+			(do_not_autoplace no)
+			(effects
+				(font
+					(size 1.27 1.27)
+				)
+			)
+		)
+		(property "LCSC Part" "C113101"
+			(at 259.08 118.11 0)
+			(hide yes)
+			(show_name no)
+			(do_not_autoplace no)
+			(effects
+				(font
+					(size 1.27 1.27)
+				)
+			)
+		)
+		(pin "2"
+		)
+		(pin "1"
+		)
+		(instances
+			(project "ZumoRobot"
+				(path "/b3437995-bb94-4c2f-9ed8-b1af477fe956/bbae36a6-1608-41fb-8b94-fa07ee9e7141"
+					(reference "L2")
+					(unit 1)
+				)
+			)
+		)
+	)
+	(symbol
 		(lib_id "EasyEDA:SS24-SMB")
 		(at 170.18 100.33 0)
@@
 					(unit 1)
 				)
-			)
-		)
-	)
-	(symbol
-		(lib_id "Snapeda:MDMK2020T2R2MM")
-		(at 259.715 107.315 0)
-		(mirror y)
-		(unit 1)
-		(body_style 1)
-		(exclude_from_sim no)
-		(in_bom no)
-		(on_board yes)
-		(in_pos_files yes)
-		(dnp no)
-		(property "Reference" "L1"
-			(at 258.445 93.853 0)
-			(show_name no)
-			(do_not_autoplace no)
-			(effects
-				(font
-					(size 1.524 1.524)
-				)
-				(justify left)
-			)
-		)
-		(property "Value" "MDMK2020T2R2MM"
-			(at 267.843 96.393 0)
-			(show_name no)
-			(do_not_autoplace no)
-			(effects
-				(font
-					(size 1.524 1.524)
-				)
-				(justify left)
-			)
-		)
-		(property "Footprint" "Snapeda:IND_MDMK2020T1R0MM_TAY"
-			(at 258.445 100.9649 0)
-			(hide yes)
-			(show_name no)
-			(do_not_autoplace no)
-			(effects
-				(font
-					(size 1.27 1.27)
-				)
-				(justify left)
-			)
-		)
-		(property "Datasheet" "MDMK2020T2R2MM"
-			(at 258.445 103.5049 0)
-			(hide yes)
-			(show_name no)
-			(do_not_autoplace no)
-			(effects
-				(font
-					(size 1.27 1.27)
-				)
-				(justify left)
-			)
-		)
-		(property "Description" ""
-			(at 259.715 107.315 0)
-			(hide yes)
-			(show_name no)
-			(do_not_autoplace no)
-			(effects
-				(font
-					(size 1.27 1.27)
-				)
-			)
-		)
-		(pin "1"
-		)
-		(pin "2"
-		)
-		(instances
-			(project "ZumoRobot"
-				(path "/b3437995-bb94-4c2f-9ed8-b1af477fe956/bbae36a6-1608-41fb-8b94-fa07ee9e7141"
-					(reference "L1")
-					(unit 1)
-				)

Commit message: terminada
Parts:
- renumbered L2 to L1, R11 to R12, U2 to U4
Changed lines of the file:
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@@
 		(dnp no)
 		(fields_autoplaced yes)
-		(property "Reference" "#PWR025"
+		(property "Reference" "#PWR026"
 			(at 203.2 101.6 0)
 			(hide yes)
@@
 			(project "ZumoRobot"
 				(path "/b3437995-bb94-4c2f-9ed8-b1af477fe956/bbae36a6-1608-41fb-8b94-fa07ee9e7141"
-					(reference "#PWR025")
+					(reference "#PWR026")
 					(unit 1)
 				)
@@
 		(in_pos_files yes)
 		(dnp no)
-		(property "Reference" "R11"
+		(property "Reference" "R12"
 			(at 278.13 99.06 90)
 			(show_name no)
@@
 			(project "ZumoRobot"
 				(path "/b3437995-bb94-4c2f-9ed8-b1af477fe956/bbae36a6-1608-41fb-8b94-fa07ee9e7141"
-					(reference "R11")
+					(reference "R12")
 					(unit 1)
 				)
@@
 		(dnp no)
 		(fields_autoplaced yes)
-		(property "Reference" "#PWR026"
+		(property "Reference" "#PWR027"
 			(at 203.2 139.7 0)
 			(hide yes)
@@
 			(project "ZumoRobot"
 				(path "/b3437995-bb94-4c2f-9ed8-b1af477fe956/bbae36a6-1608-41fb-8b94-fa07ee9e7141"
-					(reference "#PWR026")
+					(reference "#PWR027")
 					(unit 1)
 				)
@@
 		(dnp no)
 		(fields_autoplaced yes)
-		(property "Reference" "#PWR029"
+		(property "Reference" "#PWR030"
 			(at 287.02 123.19 0)
 			(hide yes)
@@
 			(project "ZumoRobot"
 				(path "/b3437995-bb94-4c2f-9ed8-b1af477fe956/bbae36a6-1608-41fb-8b94-fa07ee9e7141"
-					(reference "#PWR029")
+					(reference "#PWR030")
 					(unit 1)
 				)
@@
 		(dnp no)
 		(fields_autoplaced yes)
-		(property "Reference" "U2"
+		(property "Reference" "U4"
 			(at 229.87 92.71 0)
 			(show_name no)
@@
 			(project "ZumoRobot"
 				(path "/b3437995-bb94-4c2f-9ed8-b1af477fe956/bbae36a6-1608-41fb-8b94-fa07ee9e7141"
-					(reference "U2")
+					(reference "U4")
 					(unit 1)
 				)
@@
 		(dnp no)
 		(fields_autoplaced yes)
-		(property "Reference" "#PWR027"
+		(property "Reference" "#PWR028"
 			(at 227.33 129.54 0)
 			(hide yes)
@@
 			(project "ZumoRobot"
 				(path "/b3437995-bb94-4c2f-9ed8-b1af477fe956/bbae36a6-1608-41fb-8b94-fa07ee9e7141"
-					(reference "#PWR027")
+					(reference "#PWR028")
 					(unit 1)
 				)
@@
 		(dnp no)
 		(fields_autoplaced yes)
-		(property "Reference" "#PWR028"
+		(property "Reference" "#PWR029"
 			(at 287.02 82.55 0)
 			(hide yes)
@@
 			(project "ZumoRobot"
 				(path "/b3437995-bb94-4c2f-9ed8-b1af477fe956/bbae36a6-1608-41fb-8b94-fa07ee9e7141"
-					(reference "#PWR028")
+					(reference "#PWR029")
 					(unit 1)
 				)
@@
 		(dnp no)
 		(fields_autoplaced yes)
-		(property "Reference" "L2"
+		(property "Reference" "L1"
 			(at 259.05 93.98 0)
 			(show_name no)
@@
 			(project "ZumoRobot"
 				(path "/b3437995-bb94-4c2f-9ed8-b1af477fe956/bbae36a6-1608-41fb-8b94-fa07ee9e7141"
-					(reference "L2")
-					(unit 1)
-				)
+					(reference "L1")
+					(unit 1)
+				)

Commit message: commit final
Parts:
- U4: LCSC Part (none) -> C59873; now in the parts list
Other:
- moved on the sheet: D6
Changed lines of the file:
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@@
 	(wire
 		(pts
-			(xy 175.26 100.33) (xy 203.2 100.33)
+			(xy 193.04 100.33) (xy 203.2 100.33)
 		)
 		(stroke
@@
 	(wire
 		(pts
-			(xy 156.21 100.33) (xy 165.1 100.33)
+			(xy 156.21 100.33) (xy 182.88 100.33)
 		)
 		(stroke
@@
 		(body_style 1)
 		(exclude_from_sim no)
-		(in_bom no)
+		(in_bom yes)
 		(on_board yes)
 		(in_pos_files yes)
@@
 		)
 		(property "Description" "500mA Step-Down Converter with DCS-Control, fixed 3.3V output, 3-17V input voltage, WSON-8"
+			(at 229.87 107.95 0)
+			(hide yes)
+			(show_name no)
+			(do_not_autoplace no)
+			(effects
+				(font
+					(size 1.27 1.27)
+				)
+			)
+		)
+		(property "LCSC Part" "C59873"
 			(at 229.87 107.95 0)
 			(hide yes)
@@
 	(symbol
 		(lib_id "EasyEDA:SS24-SMB")
-		(at 170.18 100.33 0)
+		(at 187.96 100.33 0)
 		(mirror y)
 		(unit 1)
@@
 		(fields_autoplaced yes)
 		(property "Reference" "D6"
-			(at 170.18 93.98 0)
+			(at 187.96 93.98 0)
 			(show_name no)
 			(do_not_autoplace no)
@@
 		)
 		(property "Value" "SS24-SMB"
-			(at 170.18 96.52 0)
+			(at 187.96 96.52 0)
 			(show_name no)
 			(do_not_autoplace no)
@@
 		)
 		(property "Footprint" "EasyEDA:SMB_L4.3-W3.6-LS5.3-RD"
-			(at 170.18 107.95 0)
+			(at 187.96 107.95 0)
 			(hide yes)
 			(show_name no)
@@
 		)
 		(property "Datasheet" "https://www.lcsc.com/datasheet/C908683.pdf"
-			(at 170.18 110.49 0)
+			(at 187.96 110.49 0)
 			(hide yes)
 			(show_name no)
@@
 		)
 		(property "Description" ""
-			(at 170.18 100.33 0)
+			(at 187.96 100.33 0)
 			(hide yes)
 			(show_name no)
@@
 		)
 		(property "Manufacturer" "GOODWORK(固得沃克)"
-			(at 170.18 113.03 0)
+			(at 187.96 113.03 0)
 			(hide yes)
 			(show_name no)
@@
 		)
 		(property "MPN" "SS24-SMB"
-			(at 170.18 115.57 0)
+			(at 187.96 115.57 0)
 			(hide yes)
 			(show_name no)
@@
 		)
 		(property "LCSC Part" "C908683"
-			(at 170.18 118.11 0)
-			(hide yes)
-			(show_name no)
+			(at 187.96 118.11 0)
+			(hide yes)
+			(show_name no)
