File: DRV8411APWR.kicad_sch (KiCad schematic)
At the start: 5 parts, among them U3 DRV8411APWPR

Commit message: avanzes
Parts:
- R12: LCSC Part (none) -> C122538
Changed lines of the file:
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@@
+			)
+		)
+		(property "LCSC Part" "C122538"
+			(at 135.89 100.33 0)
+			(hide yes)
+			(show_name no)
+			(do_not_autoplace no)
+			(effects
+				(font
+					(size 1.27 1.27)
+				)
 			)
 		)

Commit message: terminada
Parts:
- renumbered R12 to R13, R13 to R14, U3 to U5
Changed lines of the file:
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@@
 		(in_pos_files yes)
 		(dnp no)
-		(property "Reference" "#PWR034"
+		(property "Reference" "#PWR035"
 			(at 217.17 102.87 0)
 			(hide yes)
@@
 			(project "ZumoRobot"
 				(path "/b3437995-bb94-4c2f-9ed8-b1af477fe956/7af026f4-cd24-461f-ad82-ec197bdc255a"
-					(reference "#PWR034")
+					(reference "#PWR035")
 					(unit 1)
 				)
@@
 		(dnp no)
 		(fields_autoplaced yes)
-		(property "Reference" "#PWR033"
+		(property "Reference" "#PWR034"
 			(at 195.58 133.35 0)
 			(hide yes)
@@
 			(project "ZumoRobot"
 				(path "/b3437995-bb94-4c2f-9ed8-b1af477fe956/7af026f4-cd24-461f-ad82-ec197bdc255a"
-					(reference "#PWR033")
+					(reference "#PWR034")
 					(unit 1)
 				)
@@
 		(dnp no)
 		(fields_autoplaced yes)
-		(property "Reference" "#PWR031"
+		(property "Reference" "#PWR032"
 			(at 135.89 99.06 0)
 			(hide yes)
@@
 			(project "ZumoRobot"
 				(path "/b3437995-bb94-4c2f-9ed8-b1af477fe956/7af026f4-cd24-461f-ad82-ec197bdc255a"
-					(reference "#PWR031")
+					(reference "#PWR032")
 					(unit 1)
 				)
@@
 		(dnp no)
 		(fields_autoplaced yes)
-		(property "Reference" "#PWR032"
+		(property "Reference" "#PWR033"
 			(at 176.53 87.63 0)
 			(hide yes)
@@
 			(project "ZumoRobot"
 				(path "/b3437995-bb94-4c2f-9ed8-b1af477fe956/7af026f4-cd24-461f-ad82-ec197bdc255a"
-					(reference "#PWR032")
+					(reference "#PWR033")
 					(unit 1)
 				)
@@
 		(in_pos_files yes)
 		(dnp no)
-		(property "Reference" "U3"
+		(property "Reference" "U5"
 			(at 198.12 87.63 0)
 			(show_name no)
@@
 			(project "ZumoRobot"
 				(path "/b3437995-bb94-4c2f-9ed8-b1af477fe956/7af026f4-cd24-461f-ad82-ec197bdc255a"
-					(reference "U3")
+					(reference "U5")
 					(unit 1)
 				)
@@
 		(dnp no)
 		(fields_autoplaced yes)
-		(property "Reference" "R12"
+		(property "Reference" "R13"
 			(at 138.43 99.0599 0)
 			(show_name no)
@@
 			(project "ZumoRobot"
 				(path "/b3437995-bb94-4c2f-9ed8-b1af477fe956/7af026f4-cd24-461f-ad82-ec197bdc255a"
-					(reference "R12")
+					(reference "R13")
 					(unit 1)
 				)
@@
 		(dnp no)
 		(fields_autoplaced yes)
-		(property "Reference" "#PWR030"
+		(property "Reference" "#PWR031"
 			(at 118.11 109.22 0)
 			(hide yes)
@@
 			(project "ZumoRobot"
 				(path "/b3437995-bb94-4c2f-9ed8-b1af477fe956/7af026f4-cd24-461f-ad82-ec197bdc255a"
-					(reference "#PWR030")
+					(reference "#PWR031")
 					(unit 1)
 				)
@@
 		(in_pos_files yes)
 		(dnp no)
-		(property "Reference" "R13"
+		(property "Reference" "R14"
 			(at 143.51 115.57 90)
 			(show_name no)
@@
 			(project "ZumoRobot"
 				(path "/b3437995-bb94-4c2f-9ed8-b1af477fe956/7af026f4-cd24-461f-ad82-ec197bdc255a"
-					(reference "R13")
-					(unit 1)
-				)
+					(reference "R14")
+					(unit 1)
+				)

Commit message: commit final
Parts:
- C10: value C_0603 -> 100 nf; LCSC Part (none) -> C14663
- C9: value CP_SMD_D6.3mm_H5.4mm -> 10uf; LCSC Part (none) -> C326595
- R13: LCSC Part C122538 -> C860067
- R14: LCSC Part (none) -> C860067
Changed lines of the file:
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@@
 			)
 		)
-		(property "Value" "CP_SMD_D6.3mm_H5.4mm"
+		(property "Value" "10uf"
 			(at 172.72 67.9449 0)
 			(show_name no)
@@
 		)
 		(property "Description" "SMD Electrolytic Capacitor, 6.3mm Diameter, 5.4mm Height, US Symbol, Alternate KiCad Library"
+			(at 176.53 67.31 0)
+			(hide yes)
+			(show_name no)
+			(do_not_autoplace no)
+			(effects
+				(font
+					(size 1.27 1.27)
+				)
+			)
+		)
+		(property "LCSC Part" "C326595"
 			(at 176.53 67.31 0)
 			(hide yes)
@@
 			)
 		)
-		(property "LCSC Part" "C122538"
+		(property "LCSC Part" "C860067"
 			(at 135.89 100.33 0)
 			(hide yes)
@@
 			)
 		)
+		(property "LCSC Part" "C860067"
+			(at 143.51 109.22 90)
+			(hide yes)
+			(show_name no)
+			(do_not_autoplace no)
+			(effects
+				(font
+					(size 1.27 1.27)
+				)
+			)
+		)
 		(pin "2"
 		)
@@
 			)
 		)
-		(property "Value" "C_0603"
+		(property "Value" "100 nf"
 			(at 186.69 68.5799 0)
 			(show_name no)
@@
 			(at 182.88 67.31 0)
 			(hide yes)
+			(show_name no)
+			(do_not_autoplace no)
+			(effects
+				(font
+					(size 1.27 1.27)
+				)
+			)
+		)
+		(property "LCSC Part" "C14663"
+			(at 182.88 67.31 0)
+			(hide yes)
